File: production/ecad/cstar-mcu.kicad_sch (KiCad schematic)
At the start: 0 parts

Commit message: UART-USB finished
UART to USB finished, mcu not done, usb connector not there
Parts:
- added C1, C2: C, symbol Device:C
- added R1, R2, R3, R4, R5, R6, R7: R, symbol Device:R
- added U1: ESP32-C6-WROOM-1U-N4, ESP32-C6-WROOM-1U-N4:XCVR_ESP32-C6-WROOM-1U-N4, symbol ESP32-C6:ESP32-C6-WROOM-1U-N4
- added U2: CP2102N-A01-GQFN28, QFN28_5X5_SIL, symbol CP2102:CP2102N-A01-GQFN28
Connections:
- new net: R6.1, U2.25 (RXD)
- new net: R1.1, U2.11 (SUSPENDb)
- new net: R5.1, U2.26 (TXD)
- new net: C1.1, R3.2, R4.2, U2.8 (VBUS)
- new net: R2.1, U2.9 (RSTb)
- new net: R7.2, U1.10 (IO8)
- new net +3.3V: C2.2, U2.6 (VDD), U2.7 (VREGIN)
- new net +3V3: R2.2, R7.1
- new net DTR: U2.28 (DTR)
- new net GND: C1.2, C2.1, R1.2, R3.1, U1.1 (GND), U1.28 (GND__1), U1.29_1 (GND__2), U1.29_2 (GND__3), U1.29_3 (GND__4), U1.29_4 (GND__5), U1.29_5 (GND__6), U1.29_6 (GND__7), U1.29_7 (GND__8), U1.29_8 (GND__9), U1.29_9 (GND__10), U2.29 (EPAD), U2.3 (GND)
- new net RTS: U2.24 (RTS)
- new net UART_RXD: R6.2, U1.24 (RXD0/GPIO17)
- new net UART_TXD: R5.2, U1.25 (TXD0/GPIO16)
- new net USB_DN: U2.5 (D-)
- new net USB_DP: U2.4 (D+)
- new net VBUSA: R4.1
- no-connect marks 0 -> 15
