File: production/ecad/MainBoard/cstar-power.kicad_sch (KiCad schematic)
At the start: 47 parts, among them IC1 LT8648SEV#PBF, J1 Conn_01x02_Pin, J2 Conn_01x02_Pin, J3 Conn_01x02_Pin, J4 XT60PW-M, U1 AZ1117IH-3.3TRG1

Commit message: Finished footprints for power schematic
Parts:
- C1, C10, C11, C12, C14, C2, C3, C4, C5, C6, C7, C8, C9: footprint (none) -> Capacitor_SMD:C_0805_2012Metric
- F1, F2, F3: footprint (none) -> Fuse:Fuse_0805_2012Metric
- J1, J2, J3: footprint (none) -> Connector_Phoenix_SPT:PhoenixContact_SPT_1.5_9-H-3.5_1x09_P3.5mm_Horizontal
- L1, L2: footprint (none) -> Inductor_SMD:L_0805_2012Metric
- R1, R10, R2, R3, R4, R5, R6, R7, R8, R9: footprint (none) -> Resistor_SMD:R_0805_2012Metric
- TP1, TP2, TP3, TP4, TP5, TP6, TP7: footprint (none) -> TestPoint:TestPoint_Pad_D2.0mm
