File: production/ecad/MainBoard/cstar-lidar.kicad_sch (KiCad schematic)
At the start: 3 parts, among them J5 Conn_01x02_Pin, J6 Conn_01x02_Pin, J7 532610771

Commit message: changed the path of the footprints and changed the name of the test points
Parts:
- J7: footprint 532610771:MOLEX_532610771 -> 532610771 (2):MOLEX_532610771
Changed lines of the file:
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@@
       (effects (font (size 1.27 1.27)) (justify left))
     )
-    (property "Footprint" "532610771:MOLEX_532610771" (at 147.32 71.12 0)
+    (property "Footprint" "532610771 (2):MOLEX_532610771" (at 147.32 71.12 0)
       (effects (font (size 1.27 1.27)) (justify bottom) hide)
     )

Commit message: footprint assignments
Parts:
- J7: footprint 532610771 (2):MOLEX_532610771 -> CSTAR-MainBoard-Footprints:MOLEX_532610771
Changed lines of the file:
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@@
       (effects (font (size 1.27 1.27)) (justify left))
     )
-    (property "Footprint" "532610771 (2):MOLEX_532610771" (at 147.32 71.12 0)
+    (property "Footprint" "CSTAR-MainBoard-Footprints:MOLEX_532610771" (at 147.32 71.12 0)
       (effects (font (size 1.27 1.27)) (justify bottom) hide)
     )

Commit message: footprint assign more
Parts:
- J5, J6: footprint Connector_Phoenix_SPT:PhoenixContact_SPT_1.5_9-H-3.5_1x09_P3.5mm_Horizontal -> Connector_PinHeader_2.54mm:PinHeader_1x02_P2.54mm_Vertical
Changed lines of the file:
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@@
       (effects (font (size 1.27 1.27)) (justify left))
     )
-    (property "Footprint" "Connector_Phoenix_SPT:PhoenixContact_SPT_1.5_9-H-3.5_1x09_P3.5mm_Horizontal" (at 101.6 73.66 0)
+    (property "Footprint" "Connector_PinHeader_2.54mm:PinHeader_1x02_P2.54mm_Vertical" (at 101.6 73.66 0)
       (effects (font (size 1.27 1.27)) hide)
     )
@@
       (effects (font (size 1.27 1.27)) (justify left))
     )
-    (property "Footprint" "Connector_Phoenix_SPT:PhoenixContact_SPT_1.5_9-H-3.5_1x09_P3.5mm_Horizontal" (at 102.87 80.01 0)
+    (property "Footprint" "Connector_PinHeader_2.54mm:PinHeader_1x02_P2.54mm_Vertical" (at 102.87 80.01 0)
       (effects (font (size 1.27 1.27)) hide)
     )
