File: production/ecad/MainBoard/CSTAR.kicad_pcb (KiCad board)
At the start: 4 copper layers, 152.4 x 101.6 mm, 181 parts, among them IC1 LT8648SEV#PBF, J1 Conn_01x02_Pin, J10 Conn_01x03_Pin, J11 B4B-PH-K-S, J12 B4B-PH-K-S, J13 Conn_01x03_Pin, J14 Conn_01x03_Pin, J15 Conn_01x03_Pin, J16 Conn_01x03_Pin, J17 Ultra_4, J18 Ultra_3, J19 Ultra_2, J2 Conn_01x02_Pin, J20 RX connect, J21 Ultra_1, J22 TX connect, J23 USB_C_Receptacle_USB2.0, J24 USB_C_Receptacle_USB2.0, J26 532610771, J28 532610771, J29 Conn_01x04_Socket, J3 Conn_01x02_Pin, J30 691137710002, J4 XT60PW-M, J5 Conn_01x02_Pin, J6 Conn_01x02_Pin, J7 532610771, J8 Conn_01x03_Pin, J9 Conn_01x03_Pin, Q1 AO3400A, Q2 AO3400A, Q3 AO3400A, Q4 AO3400A, Q5 AO3400A, Q6 AO3400A, Q7 AO3400A, Q8 IRFHM9331TRPBF, SW1 SW_Push, SW2 SW_Push, SW3 SW_Push, SW4 SW_Push, U1 AZ1117IH-3.3TRG1, U2 DRV8842PWPR, U3 DRV8842PWPR, U4 TXB0104DR, U5 CP2102N-A01-GQFN28, U6 ESP32-WROOM-32UE_M113EH6400UH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, U7 TXB0104DR, U8 CP2102N-A01-GQFN28, U9 ESP32-WROOM-32UE_M113EH6400UH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, X1 B2P-VH, X2 B2P-VH

Commit message: component placement
Parts:
- removed J24: USB_C_Receptacle_USB2.0, CSTAR-MainBoard-Footprints:USBCONN-GCT_USB4105GFA
- added J25: TYPE-C-31-M-12, CSTAR-MainBoard-Footprints:HRO_TYPE-C-31-M-12, F.Cu at (53.6, 108.0)
- added J31: TYPE-C-31-M-12, CSTAR-MainBoard-Footprints:HRO_TYPE-C-31-M-12, F.Cu at (200.5, 75.8)
- J23: value USB_C_Receptacle_USB2.0 -> Conn_01x02_Pin; footprint CSTAR-MainBoard-Footprints:USBCONN-GCT_USB4105GFA -> Connector_PinHeader_2.54mm:PinHeader_1x02_P2.54mm_Vertical
- U1: footprint CSTAR-MainBoard-Footprints:TO252-2_AZ1117ID-3.3TRG1_DIO -> CSTAR-MainBoard-Footprints:SOT230P700X185-4N
- moved LED2 223.5 mm to (89.9, 145.1), turned to 90 degrees
- moved L1 215.2 mm to (82.0, 129.6), turned to 90 degrees
- moved C3 201.2 mm to (102.1, 173.5)
- moved C8 201.2 mm to (102.1, 194.3)
- moved C4 201.2 mm to (102.1, 179.1)
- moved C6 201.2 mm to (102.1, 184.7)
- moved C7 201.2 mm to (102.1, 189.7)
- moved R3 201.2 mm to (89.2, 172.0)
- moved R4 201.2 mm to (89.2, 176.4)
- moved R5 201.2 mm to (89.2, 181.1)
- moved R7 201.2 mm to (89.2, 186.7)
- moved R8 201.2 mm to (89.2, 191.3)
- moved TP2 201.2 mm to (136.1, 168.4)
- moved TP4 201.2 mm to (136.1, 174.2)
- moved C2 201.2 mm to (102.1, 167.6)
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Connections:
- U9 pad 36: 3V_echo_4 -> nRESET
- U9 pad 4: unconnected-(U9-SENSOR_VP-Pad4) -> nFAULT MOTOR 1
- U9 pad 6: nFAULT MOTOR 1 -> 3V_echo_4

Commit message: Power Component Placement
Parts:
- moved TP6 338.6 mm to (64.0, 146.3)
- moved LED4 315.7 mm to (73.2, 127.0), turned to 90 degrees
- moved TP7 293.9 mm to (107.2, 109.0)
- moved TP5 293.8 mm to (107.2, 113.0)
- moved R9 281.7 mm to (73.2, 122.9), turned to -90 degrees
- moved L2 256.8 mm to (119.4, 109.5), turned to 180 degrees
- moved C13 255.1 mm to (110.7, 109.0), turned to -90 degrees
- moved C12 251.7 mm to (113.8, 109.0), turned to -90 degrees
- moved C9 248.8 mm to (116.3, 115.6), turned to -90 degrees
- moved C11 248.0 mm to (117.3, 126.0)
- moved C26 239.8 mm to (351.7, 71.4)
- moved C28 239.8 mm to (351.7, 77.4)
- moved C29 239.8 mm to (351.7, 80.4)
- moved CR2 239.8 mm to (351.1, 105.5)
- moved J29 239.8 mm to (377.7, 75.4)
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Connections:
- R1 pad 1: Net-(J2-Pin_1) -> +5V
- R9 pad 1: Net-(J3-Pin_1) -> +12V

Commit message: fixed USBC (sorry Cat)
Connections:
- J25 pad A6: USB1_D- -> USB1_D+
- J25 pad A7: USB1_D+ -> USB1_D-
- J25 pad B6: USB1_D- -> USB1_D+
- J25 pad B7: USB1_D+ -> USB1_D-
- J31 pad A6: USB2_D- -> USB2_D+
- J31 pad A7: USB2_D+ -> USB2_D-
- J31 pad B6: USB2_D- -> USB2_D+
- J31 pad B7: USB2_D+ -> USB2_D-
Changed lines of the file:
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@@
       (net 235 "Net-(J25-CC1)") (pinfunction "CC1") (pintype "bidirectional"))
     (pad "A6" smd rect (at -0.25 -4.75 270) (size 0.3 1.14) (layers "F.Cu" "F.Paste")
-      (net 76 "USB1_D-") (pinfunction "DP1") (pintype "bidirectional"))
+      (net 77 "USB1_D+") (pinfunction "DP1") (pintype "bidirectional"))
     (pad "A7" smd rect (at 0.25 -4.75 270) (size 0.3 1.14) (layers "F.Cu" "F.Paste")
-      (net 77 "USB1_D+") (pinfunction "DN1") (pintype "bidirectional"))
+      (net 76 "USB1_D-") (pinfunction "DN1") (pintype "bidirectional"))
     (pad "A8" smd rect (at 1.25 -4.75 270) (size 0.3 1.14) (layers "F.Cu" "F.Paste")
       (net 240 "unconnected-(J25-SBU1-PadA8)") (pinfunction "SBU1") (pintype "bidirectional+no_connect"))
@@
       (net 234 "Net-(J25-CC2)") (pinfunction "CC2") (pintype "bidirectional"))
     (pad "B6" smd rect (at 0.75 -4.75 270) (size 0.3 1.14) (layers "F.Cu" "F.Paste")
-      (net 76 "USB1_D-") (pinfunction "DP2") (pintype "bidirectional"))
+      (net 77 "USB1_D+") (pinfunction "DP2") (pintype "bidirectional"))
     (pad "B7" smd rect (at -0.75 -4.75 270) (size 0.3 1.14) (layers "F.Cu" "F.Paste")
-      (net 77 "USB1_D+") (pinfunction "DN2") (pintype "bidirectional"))
+      (net 76 "USB1_D-") (pinfunction "DN2") (pintype "bidirectional"))
     (pad "B8" smd rect (at -1.75 -4.75 270) (size 0.3 1.14) (layers "F.Cu" "F.Paste")
       (net 239 "unconnected-(J25-SBU2-PadB8)") (pinfunction "SBU2") (pintype "bidirectional+no_connect"))
@@
       (net 236 "Net-(J31-CC1)") (pinfunction "CC1") (pintype "bidirectional"))
     (pad "A6" smd rect (at -0.25 -4.75 90) (size 0.3 1.14) (layers "F.Cu" "F.Paste")
-      (net 80 "USB2_D-") (pinfunction "DP1") (pintype "bidirectional"))
+      (net 81 "USB2_D+") (pinfunction "DP1") (pintype "bidirectional"))
     (pad "A7" smd rect (at 0.25 -4.75 90) (size 0.3 1.14) (layers "F.Cu" "F.Paste")
-      (net 81 "USB2_D+") (pinfunction "DN1") (pintype "bidirectional"))
+      (net 80 "USB2_D-") (pinfunction "DN1") (pintype "bidirectional"))
     (pad "A8" smd rect (at 1.25 -4.75 90) (size 0.3 1.14) (layers "F.Cu" "F.Paste")
       (net 243 "unconnected-(J31-SBU1-PadA8)") (pinfunction "SBU1") (pintype "bidirectional+no_connect"))
@@
       (net 237 "Net-(J31-CC2)") (pinfunction "CC2") (pintype "bidirectional"))
     (pad "B6" smd rect (at 0.75 -4.75 90) (size 0.3 1.14) (layers "F.Cu" "F.Paste")
-      (net 80 "USB2_D-") (pinfunction "DP2") (pintype "bidirectional"))
+      (net 81 "USB2_D+") (pinfunction "DP2") (pintype "bidirectional"))
     (pad "B7" smd rect (at -0.75 -4.75 90) (size 0.3 1.14) (layers "F.Cu" "F.Paste")
-      (net 81 "USB2_D+") (pinfunction "DN2") (pintype "bidirectional"))
+      (net 80 "USB2_D-") (pinfunction "DN2") (pintype "bidirectional"))
     (pad "B8" smd rect (at -1.75 -4.75 90) (size 0.3 1.14) (layers "F.Cu" "F.Paste")
       (net 242 "unconnected-(J31-SBU2-PadB8)") (pinfunction "SBU2") (pintype "bidirectional+no_connect"))

Commit message: "Started Layout for MOTOR IC"
Parts:
- moved C19 259.5 mm to (97.0, 79.3), turned to -90 degrees
- moved C17 254.9 mm to (97.0, 83.1), turned to 90 degrees
- moved C20 254.2 mm to (101.9, 76.2), turned to 180 degrees
- moved C18 225.8 mm to (131.1, 78.8), turned to -90 degrees
- moved C16 221.1 mm to (131.1, 82.3), turned to 90 degrees
- moved R19 169.7 mm to (91.9, 83.2), turned to 90 degrees
- moved R18 134.3 mm to (128.1, 82.3), turned to 90 degrees
- moved U3 12.8 mm to (109.4, 85.4)

Commit message: More component placement (motor controllers and jumpers)
Parts:
- moved C25 266.2 mm to (95.0, 88.0), turned to -90 degrees
- moved C23 263.3 mm to (98.5, 88.0), turned to -90 degrees
- moved C21 255.2 mm to (101.6, 88.0), turned to -90 degrees
- moved C15 238.6 mm to (114.8, 90.4), turned to -90 degrees
- moved C24 220.6 mm to (141.1, 87.8), turned to -90 degrees
- moved C22 217.6 mm to (144.9, 87.8), turned to -90 degrees
- moved R43 197.5 mm to (60.6, 238.9)
- moved R48 197.5 mm to (60.6, 244.8)
- moved R51 197.5 mm to (60.6, 253.6)
- moved U7 197.5 mm to (64.0, 217.1)
- moved R45 197.5 mm to (60.6, 241.8)
- moved R49 197.5 mm to (60.6, 247.7)
- moved R50 197.5 mm to (60.6, 250.7)
- moved R52 197.5 mm to (60.6, 256.6)
- moved R53 197.5 mm to (60.6, 259.5)
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
Commit message: more component placement!
Parts:
- added J13: Conn_01x05_Pin, Connector_PinSocket_2.54mm:PinSocket_1x05_P2.54mm_Vertical, F.Cu at (208.3, 22.9)
- added J23: USB_C_Receptacle_USB2.0, CSTAR-MainBoard-Footprints:USBCONN-GCT_USB4105GFA, F.Cu at (43.2, 106.7)
- added J24: USB_C_Receptacle_USB2.0, CSTAR-MainBoard-Footprints:USBCONN-GCT_USB4105GFA, F.Cu at (210.8, 91.4)
- added J25: Conn_01x02_Pin, Connector_PinSocket_2.54mm:PinSocket_1x02_P2.54mm_Vertical, F.Cu at (212.9, 22.9)
- added R32: 5.1k, Resistor_SMD:R_0805_2012Metric, F.Cu at (248.0, 35.6)
- added R33: 5.1k, Resistor_SMD:R_0805_2012Metric, F.Cu at (248.0, 38.5)
- added R43: 5.1k, Resistor_SMD:R_0805_2012Metric, F.Cu at (248.0, 41.5)
- added R45: 5.1k, Resistor_SMD:R_0805_2012Metric, F.Cu at (248.0, 44.4)
- C7, C8: footprint Capacitor_SMD:C_1206_3216Metric -> Capacitor_SMD:C_0805_2012Metric
- L1: footprint CSTAR-MainBoard-Footprints:L1_2.2uH -> Inductor_SMD:L_0805_2012Metric
- L2: footprint CSTAR-MainBoard-Footprints:L2_6.8uH -> Inductor_SMD:L_0805_2012Metric
- U1: footprint CSTAR-MainBoard-Footprints:SOT230P700X185-4N -> CSTAR-MainBoard-Footprints:TO252-2_AZ1117ID-3.3TRG1_DIO
- moved R43 246.0 mm to (266.7, 104.6)
- moved R45 246.0 mm to (266.7, 107.6)
- moved R48 246.0 mm to (266.7, 110.5)
- moved R49 246.0 mm to (266.7, 113.5)
- moved R50 246.0 mm to (266.7, 116.4)
- moved R51 246.0 mm to (266.7, 119.4)
- moved R52 246.0 mm to (266.7, 122.3)
- moved R53 246.0 mm to (266.7, 125.3)
- moved U7 171.6 mm to (175.3, 86.4), turned to 90 degrees
- moved R41 143.1 mm to (194.0, 106.7)
- moved R40 143.1 mm to (194.0, 103.9)
- moved U4 127.6 mm to (135.8, 118.1), turned to 180 degrees
- moved J22 58.0 mm to (167.6, 106.7)
- moved C26 48.7 mm to (303.8, 80.3)
- moved C27 48.7 mm to (303.8, 83.3)
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Connections:
- net nSLEEP renamed SCL
- J26 pad 4: SDTO -> I2S_D2
- J26 pad 5: LRCK -> I2S_CLK
- J26 pad 6: MCLK -> I2S_CMD
- J26 pad 7: BICK -> I2S_D0
- J28 pad 4: SDTO2 -> I2S_D3
- J28 pad 5: LRCK2 -> I2S_CLK
- J28 pad 6: MCLK2 -> I2S_CMD
- J28 pad 7: BICK2 -> I2S_D1
- R1 pad 1: +5V -> Net-(J2-Pin_1)
- R9 pad 1: +12V -> Net-(J3-Pin_1)
- TP10 pad 1: /CSTAR-Drive/IN1_MOTOR_1 -> IN1_MOTOR_1
- TP11 pad 1: /CSTAR-Drive/IN2_MOTOR_1 -> IN2_MOTOR_1
- TP12 pad 1: /CSTAR-Drive/IN1_MOTOR_2 -> IN1_MOTOR_2
- TP13 pad 1: /CSTAR-Drive/IN2_MOTOR_2 -> IN2_MOTOR_2
- U2 pad 16: /CSTAR-Drive/nRESET -> RST
- U2 pad 20: /CSTAR-Drive/IN2_MOTOR_1 -> IN2_MOTOR_1
- U2 pad 21: /CSTAR-Drive/IN1_MOTOR_1 -> IN1_MOTOR_1
- U3 pad 16: /CSTAR-Drive/nRESET -> RST
- U3 pad 20: /CSTAR-Drive/IN2_MOTOR_2 -> IN2_MOTOR_2
- U3 pad 21: /CSTAR-Drive/IN1_MOTOR_2 -> IN1_MOTOR_2
- U4 pad 8: Net-(U4-OE) -> unconnected-(U4-OE-Pad8)
- U7 pad 8: Net-(U7-OE) -> unconnected-(U7-OE-Pad8)
- U9 pad 14: OUT1 MOTOR 2 -> IN1_MOTOR_2
- U9 pad 24: OUT2 MOTOR 1 -> IN2_MOTOR_1
- U9 pad 26: OUT1 MOTOR 1 -> IN1_MOTOR_1
- U9 pad 29: OUT2 MOTOR 2 -> IN2_MOTOR_2
- U9 pad 36: nRESET -> 3V_echo_4
- U9 pad 6: 3V_echo_4 -> nFAULT MOTOR 1
Other:
- board size 152.4 x 101.6 mm -> 152.4 x 127 mm

Commit message: reannotated to fix sch
Parts:
- removed the J24 at (210.8, 91.4)
- C7, C8: footprint Capacitor_SMD:C_0805_2012Metric -> Capacitor_SMD:C_1206_3216Metric
- J23: value USB_C_Receptacle_USB2.0 -> Conn_01x02_Pin; footprint CSTAR-MainBoard-Footprints:USBCONN-GCT_USB4105GFA -> Connector_PinHeader_2.54mm:PinHeader_1x02_P2.54mm_Vertical
- L1: footprint Inductor_SMD:L_0805_2012Metric -> CSTAR-MainBoard-Footprints:L1_2.2uH
- L2: footprint Inductor_SMD:L_0805_2012Metric -> CSTAR-MainBoard-Footprints:L2_6.8uH
- U1: footprint CSTAR-MainBoard-Footprints:TO252-2_AZ1117ID-3.3TRG1_DIO -> CSTAR-MainBoard-Footprints:SOT230P700X185-4N
- moved J23 261.3 mm to (294.6, 35.6), turned to 0 degrees
- moved R43 48.8 mm to (218.5, 96.5)
- moved R45 48.8 mm to (218.5, 99.4)
- moved R48 48.8 mm to (218.5, 102.4)
- moved R49 48.8 mm to (218.5, 105.3)
- moved R50 48.8 mm to (218.5, 108.3)
- moved R51 48.8 mm to (218.5, 111.2)
- moved R52 48.8 mm to (218.5, 114.2)
- moved R53 48.8 mm to (218.5, 117.1)
- renumbered J25 to J24
Connections:
- R1 pad 1: Net-(J2-Pin_1) -> +5V
- R9 pad 1: Net-(J3-Pin_1) -> +12V
- U4 pad 8: unconnected-(U4-OE-Pad8) -> Net-(U4-OE)
- U7 pad 8: unconnected-(U7-OE-Pad8) -> Net-(U7-OE)
- U9 pad 14: IN1_MOTOR_2 -> OUT1 MOTOR 2
- U9 pad 24: IN2_MOTOR_1 -> OUT2 MOTOR 1
- U9 pad 26: IN1_MOTOR_1 -> OUT1 MOTOR 1
- U9 pad 29: IN2_MOTOR_2 -> OUT2 MOTOR 2
- U9 pad 36: 3V_echo_4 -> RST
- U9 pad 6: nFAULT MOTOR 1 -> 3V_echo_4

Commit message: MORE LAYOUT and some schematic changes
Parts:
- removed the J23 at (128.1, 142.9)
- removed R32 (x2), R33 (x2): 5.1k, Resistor_SMD:R_0805_2012Metric
- removed the R43 at (287.9, 141.0)
- removed the R43 at (248.0, 41.5)
- removed the R45 at (248.0, 44.4)
- removed the R45 at (218.5, 99.4)
- removed the R45 at (287.9, 146.9)
- added R45: 10k, Resistor_SMD:R_0805_2012Metric, F.Cu at (118.9, 142.5)
- moved TP17 282.8 mm to (62.7, 61.2)
- moved J29 278.2 mm to (77.4, 201.2), turned to 180 degrees
- moved TP16 271.2 mm to (73.9, 60.5)
- moved TP10 267.1 mm to (68.6, 71.4)
- moved TP21 266.9 mm to (82.7, 60.2)
- moved TP11 265.1 mm to (72.1, 71.6)
- moved TP-VGSW1 265.0 mm to (77.5, 190.2)
- moved TP19 258.3 mm to (88.6, 60.5)
- moved C30 257.6 mm to (53.1, 115.3)
- moved C31 257.0 mm to (53.1, 113.3)
- moved TP22 253.2 mm to (77.5, 195.1)
- moved C38 241.9 mm to (82.3, 192.0), turned to -90 degrees
- moved CR1 240.8 mm to (68.1, 59.7)
- moved C29 234.1 mm to (70.1, 76.5), turned to 90 degrees
- moved C26 229.4 mm to (82.5, 141.0), turned to 90 degrees
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Connections:
- C30 pad 1: +3V3 -> GND
- C30 pad 2: Net-(U6-3V3) -> +3V3
- C31 pad 1: +3V3 -> GND
- C31 pad 2: Net-(U6-3V3) -> +3V3
- C36 pad 1: +3V3 -> GND
- C36 pad 2: Net-(U9-3V3) -> +3V3
- C37 pad 1: +3V3 -> GND
- C37 pad 2: Net-(U9-3V3) -> +3V3
- Q5 pad 1: /CSTAR-IO/RGB_Red_Control -> RGB_Red_Control
- Q6 pad 1: /CSTAR-IO/RBG_Green_Control -> RGB_Green_Control
- Q7 pad 1: /CSTAR-IO/RGB_Blue_Control -> RGB_Blue_Control
- U6 pad 2: Net-(U6-3V3) -> +3V3
- U9 pad 2: Net-(U9-3V3) -> +3V3
Other:
- board size 152.4 x 127 mm -> 152.4 x 152.4 mm
