File: PCB_Rev1/Main_Board_Rev1/cstar-power.kicad_sch (KiCad schematic)
At the start: 0 parts

Commit message: Motor Drive Circuit
L298N motor driver and motor connections added
Other:
- note added: "Power 24V Battery"
Changed lines of the file:
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@@
 	(generator_version "8.0")
 	(paper "A4")
+	(text "Power 24V Battery\n"
+		(exclude_from_sim no)
+		(at 135.255 -6.35 0)
+		(effects
+			(font
+				(size 6 6)
+				(bold yes)
+			)
+			(justify left bottom)
+		)
+	)
 )
