File: PCB_Rev1/Main_Board_Rev1/cstar-lidar.kicad_sch (KiCad schematic)
At the start: 0 parts

Commit message: Update cstar-lidar.kicad_sch for RPi
Parts:
- added J3: 532610771, CSTAR-MainBoard-Footprints:MOLEX_532610771, symbol 532610771:532610771
Connections:
- new net +5V: J3.1, J3.5
- new net GND: J3.3, J3.4, J3.S1 (SHIELD1), J3.S2 (SHIELD2)
- new net GPIO14: J3.6
- new net GPIO15: J3.7
- new net GPIO17: J3.2
Other:
- note added: "Lidar Connector"
